Commit message: code loi phan gazebo, luu tam de chinh sua file package.xml va cmake

File: src/mobile_robot/urdf/mobile_robot.urdf (robot description, URDF)
Before this commit: robot mobile_robot, 7 links, 6 joints
Links:
- added link dummy
Joints:
- added joint dummy_joint: type fixed, parent dummy, child base_link, origin xyz=0 0 0.02 rpy=0 0 0

Commit message: gazebo ok

File: src/mobile_robot/urdf/mobile_robot.urdf (robot description, URDF)
Before this commit: robot mobile_robot, 8 links, 7 joints
Links:
- removed link caster_back
- removed link caster_back_wheel
- removed link caster_front
- removed link caster_front_wheel
- removed link dummy
- added link base_footprint, mass 0.0001; visual box size=0.001 0.001 0.001
- link base_link: mass 1.0999 -> 1.1834
- link left_wheel: geometry collision mesh filename=package://mobile_robot/meshes/left_wheel.STL; visual mesh filename=package://mobile_robot/meshes/left_wheel.STL
- link right_wheel: geometry collision mesh filename=package://mobile_robot/meshes/right_wheel.STL; visual mesh filename=package://mobile_robot/meshes/right_wheel.STL
Joints:
- removed joint caster_back_joint
- removed joint caster_back_wheel_joint
- removed joint caster_front_joint
- removed joint caster_front_wheel_joint
- removed joint dummy_joint
- added joint base_footprint_joint: type fixed, parent base_footprint, child base_link, origin xyz=0 0 0.04 rpy=0 0 0
- joint left_wheel_joint: limit effort=0.1 velocity=10 -> effort=0.5 velocity=5; origin xyz=-0.102 0 0.02 rpy=-1.5708 0 3.1416 -> xyz=-0.11958 0.00072065 0.029 rpy=-1.5888 0 3.1416
- joint right_wheel_joint: limit effort=0.1 velocity=10 -> effort=0.5 velocity=5; origin xyz=0.102 0 0.02 rpy=-1.5708 0 3.1416 -> xyz=0.11958 0.00072065 0.029 rpy=-1.5888 0 3.1416

Commit message: da them laser scanner nhung ko thay hien thi tren rviz

File: src/mobile_robot/urdf/mobile_robot.urdf (robot description, URDF)
Before this commit: robot mobile_robot, 4 links, 3 joints
Links:
- added link laser_link, mass 0.5; collision box size=0.1 0.1 0.1; visual mesh filename=package://mobile_robot/meshes/hokuyo.dae
Joints:
- added joint laser_joint: type fixed, parent base_link, child laser_link, origin xyz=0 0 0.095 rpy=0 0 1.57079, axis 0 1 0

Commit message: Da chay duoc laser tren rviz

File: src/mobile_robot/urdf/mobile_robot.urdf (robot description, URDF)
Before this commit: robot mobile_robot, 5 links, 4 joints
Links:
- link laser_link: mass 0.5 -> 0.270; geometry collision box size=0.058 0.058 0.087; visual mesh filename=package://mobile_robot/meshes/hokuyo.dae
Joints:
- joint laser_joint: origin xyz=0 0 0.095 rpy=0 0 1.57079 -> xyz=0 0 0.1 rpy=0 0 1.57079

Commit message: Da xay dung duoc map

File: src/mobile_robot/urdf/mobile_robot.urdf (robot description, URDF)
Before this commit: robot mobile_robot, 5 links, 4 joints
Links:
- link base_footprint: mass 0.0001 -> None; geometry 
